File: Model S/v1.brd (EAGLE design)
At the start: 39.8 x 39.8 mm, 45 parts, among them IC1 MCP1703CB, Q2 FDN360P

Commit message: Finished Sensor Node Model S, created gerbers
Parts:
- added PORT_A: (no value), SparkFun-Connectors:AVR_ICSP
- added U$2: (no value), SparkFun-Aesthetics:OSHW-LOGO-M
- added U$3: (no value), mystuff:PI_XS
- added U1: (no value), Seeed-OPL-ic:LQFP64-0.5-10X10MM
- JP3: device SparkFun-Connectors:AVR_ICSP -> SparkFun-Connectors:1X01NS-KIT
- U$1: device Seeed-OPL-ic:LQFP64-0.5-10X10MM -> mystuff:PI
- moved JP3 11.3 mm to (14.8, 5.95), turned to 0 degrees
- moved U$1 3.58 mm to (18.1, 18.8)
- renumbered CN1 to VIN, D2 to LED2, D3 to LED1, J2 to USB, JP1 to SWD, JP2 to SERIAL_1, JP4 to PORT_B, JP5 to SPI_2, JP7 to SERIAL_2, SW1 to BTN1, SW2 to RESET
Connections:
- net A0: now also U1.14; no longer U$1.14
- net A1: now also PORT_A.4, U1.15; no longer JP3.4, U$1.15
- net A10: now also U1.43; no longer U$1.43
- net A15: now also U1.50; no longer U$1.50
- net A2: now also U1.16; no longer U$1.16
- net A3: now also U1.17; no longer U$1.17
- net A4: now also PORT_A.6, U1.20; no longer JP3.6, U$1.20
- net A5: now also PORT_A.9, U1.21; no longer JP3.9, U$1.21
- net A6: now also PORT_A.8, U1.22; no longer JP3.8, U$1.22
- net A7: now also PORT_A.10, U1.23; no longer JP3.10, U$1.23
- net A8: now also U1.41; no longer U$1.41
- net B0: now also U1.26; no longer U$1.26
- net B1: now also U1.27; no longer U$1.27
- net B10: now also U1.29; no longer U$1.29
- net B12: now also U1.33; no longer U$1.33
- net B13: now also U1.34; no longer U$1.34
- net B14: now also U1.35; no longer U$1.35
- net B15: now also U1.36; no longer U$1.36
- net B2: now also JP3.1, U1.28; no longer U$1.28
- net B3: now also U1.55; no longer U$1.55
- net B4: now also U1.56; no longer U$1.56
- net B5: now also U1.57; no longer U$1.57
- net B6: now also U1.58; no longer U$1.58
- net B7: now also U1.59; no longer U$1.59
- net B8: now also PORT_A.5, U1.61; no longer JP3.5, U$1.61
- net B9: now also PORT_A.7, U1.62; no longer JP3.7, U$1.62
- net BOOT0: now also U1.60; no longer U$1.60
- net C0: now also U1.8; no longer U$1.8
- net C1: now also U1.9; no longer U$1.9
- net C10: now also U1.51; no longer U$1.51
- net C11: now also U1.52; no longer U$1.52
- net C12: now also U1.53; no longer U$1.53
- net C13: now also U1.2; no longer U$1.2
- net C2: now also U1.10; no longer U$1.10
- net C3: now also U1.11; no longer U$1.11
- net C4: now also U1.24; no longer U$1.24
- net C5: now also U1.25; no longer U$1.25
- net C6: now also U1.37; no longer U$1.37
- net C7: now also U1.38; no longer U$1.38
- net C8: now also U1.39; no longer U$1.39
- net C9: now also U1.40; no longer U$1.40
- net D2: now also U1.54; no longer U$1.54
- net GND: now also PORT_A.1, U1.12, U1.18, U1.31, U1.47, U1.63; no longer JP3.1, U$1.12, U$1.18, U$1.31, U$1.47, U$1.63
- net INT: now also PORT_A.2; no longer JP3.2
- net N$1: now also U1.3; no longer U$1.3
- net N$2: now also U1.30; no longer U$1.30
- net N$3: now also U1.4; no longer U$1.4
- net N$4: now also U1.5; no longer U$1.5
- net N$5: now also U1.6; no longer U$1.6
- net N$6: now also U1.44; no longer U$1.44
- net N$7: now also U1.45; no longer U$1.45
- net NRST: now also U1.7; no longer U$1.7
- net SWCLK: now also U1.49; no longer U$1.49
- net SWDIO: now also U1.46; no longer U$1.46
- net VDD: now also PORT_A.3, U1.1, U1.13, U1.19, U1.32, U1.48, U1.64; no longer JP3.3, U$1.1, U$1.13, U$1.19, U$1.32, U$1.48, U$1.64
- net VUSB: now also U1.42; no longer U$1.42
Routing:
- net B2: track 9.18 -> 17.2 mm
- net INT: track 101.7 -> 97.8 mm
- net GND: track 106.6 -> 107.7 mm, vias 9 -> 10
Other:
- outline, holes or cut-outs redrawn
- board text added: "- VIN +"
- board text added: "A0"
- board text added: "A1"
- board text added: "A4"
- board text added: "A5"
- board text added: "A6"
- board text added: "A7"
- board text added: "B10"
- board text added: "B3"
- board text added: "B8"
- board text added: "B9"
- board text added: "BOOT0"
- board text added: "BOOT1"
- board text added: "C2"
- board text added: "C3"
- board text added: "G"
- board text added: "NRST"
- board text added: "RX"
- board text added: "SWCLK"
- board text added: "SWDIO"
- board text added: "TX"
- board text added: "V"
- board text added: "Wireless Sensor Node S v1.0"
- board text added: "www.addictedtopi.com"
