File: Model S/v1.sch (EAGLE design)
At the start: 45 parts, among them IC1 MCP1703CB, Q2 FDN360P

Commit message: Finished Sensor Node Model S, created gerbers
Parts:
- added PORT_A: (no value), SparkFun-Connectors:M05X2PTH
- JP3: device SparkFun-Connectors:M05X2PTH -> SparkFun-Connectors:M01NOSILK-KIT
- renumbered CN1 to VIN, D2 to LED2, D3 to LED1, J2 to USB, JP1 to SWD, JP2 to SERIAL_1, JP4 to PORT_B, JP5 to SPI_2, JP7 to SERIAL_2, SW1 to BTN1, SW2 to RESET, U$1 to U1
Connections:
- net A1: now also PORT_A.4; no longer JP3.4
- net A4: now also PORT_A.6; no longer JP3.6
- net A5: now also PORT_A.9; no longer JP3.9
- net A6: now also PORT_A.8; no longer JP3.8
- net A7: now also PORT_A.10; no longer JP3.10
- net B2: now also JP3.1
- net B8: now also PORT_A.5; no longer JP3.5
- net B9: now also PORT_A.7; no longer JP3.7
- net GND: now also PORT_A.1; no longer JP3.1
- net INT: now also PORT_A.2; no longer JP3.2
- net VDD: now also PORT_A.3; no longer JP3.3
